File: Hardware/JsonPaper.kicad_sch (KiCad schematic)
At the start: 7 parts, among them J1 PICO-9, SW1 WS-TATV, U1 ESP32-C5-DevKit

Commit message: Add BOM
Parts:
- H1, H2, H3, H4: Symbol (none) -> ${SYMBOL_LIBRARY}:${SYMBOL_NAME}; now left out of the parts list
- J1, SW1, U1: Symbol (none) -> ${SYMBOL_LIBRARY}:${SYMBOL_NAME}
Connections:
- no-connect marks 19 -> 18
Changed lines of the file:
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@@
-	)
-	(no_connect
-		(at 67.31 135.89)
 	)
 	(no_connect
@@
 		(body_style 1)
 		(exclude_from_sim no)
-		(in_bom yes)
+		(in_bom no)
 		(on_board yes)
 		(in_pos_files yes)
@@
 			)
 		)
+		(property "Symbol" "${SYMBOL_LIBRARY}:${SYMBOL_NAME}"
+			(at 91.44 123.19 0)
+			(hide yes)
+			(show_name no)
+			(do_not_autoplace no)
+			(effects
+				(font
+					(size 1.27 1.27)
+				)
+			)
+		)
 		(pin "1"
 		)
@@
 		(body_style 1)
 		(exclude_from_sim no)
-		(in_bom yes)
+		(in_bom no)
 		(on_board yes)
 		(in_pos_files yes)
@@
 		)
 		(property "ItemNo" "503003"
+			(at 91.44 114.3 0)
+			(hide yes)
+			(show_name no)
+			(do_not_autoplace no)
+			(effects
+				(font
+					(size 1.27 1.27)
+				)
+			)
+		)
+		(property "Symbol" "${SYMBOL_LIBRARY}:${SYMBOL_NAME}"
 			(at 91.44 114.3 0)
 			(hide yes)
@@
 			)
 		)
+		(property "Symbol" "${SYMBOL_LIBRARY}:${SYMBOL_NAME}"
+			(at 205.74 120.65 0)
+			(hide yes)
+			(show_name no)
+			(do_not_autoplace no)
+			(effects
+				(font
+					(size 1.27 1.27)
+				)
+			)
+		)
 		(pin "1"
 		)
@@
 			)
 		)
+		(property "Symbol" "${SYMBOL_LIBRARY}:${SYMBOL_NAME}"
+			(at 189.23 81.28 90)
+			(hide yes)
+			(show_name no)
+			(do_not_autoplace no)
+			(effects
+				(font
+					(size 1.27 1.27)
+				)
+			)
+		)
 		(pin "1"
 		)
@@
 		(body_style 1)
 		(exclude_from_sim no)
-		(in_bom yes)
+		(in_bom no)
 		(on_board yes)
 		(in_pos_files yes)
@@
 			)
 		)
+		(property "Symbol" "${SYMBOL_LIBRARY}:${SYMBOL_NAME}"
+			(at 81.28 114.3 0)
+			(hide yes)
+			(show_name no)
+			(do_not_autoplace no)
+			(effects
+				(font
+					(size 1.27 1.27)
+				)
+			)
+		)
 		(pin "1"
 		)
@@
 		(body_style 1)
 		(exclude_from_sim no)
-		(in_bom yes)
+		(in_bom no)
 		(on_board yes)
 		(in_pos_files yes)
@@
 		)
 		(property "ItemNo" "503003"
+			(at 81.28 123.19 0)
+			(hide yes)
+			(show_name no)
+			(do_not_autoplace no)
+			(effects
+				(font
+					(size 1.27 1.27)
+				)
+			)
+		)
+		(property "Symbol" "${SYMBOL_LIBRARY}:${SYMBOL_NAME}"
 			(at 81.28 123.19 0)
 			(hide yes)
@@
 			(at 146.05 57.15 0)
 			(hide yes)
+			(show_name no)
+			(do_not_autoplace no)
+			(effects
+				(font
+					(size 1.27 1.27)
+				)
+			)
+		)
+		(property "Symbol" "${SYMBOL_LIBRARY}:${SYMBOL_NAME}"
+			(at 146.05 57.15 0)
+			(hide yes)
